File: esp12breakout2.kicad_pcb (KiCad board)
At the start: 2 copper layers, 26.7 x 44.5 mm, 15 parts, among them P1 CONN_01X08, P2 CONN_01X08, P3 FT232_3V3, SW1 reset, SW2 program

Commit message: ...
Parts:
- added ?: , initials:initials, F.Cu at (232.2, 107.2)
- added ?: , initials:initials, F.Cu at (194.6, 116.8)
Routing:
- net /TX: track 47.2 -> 49.6 mm
- net /RX: track 56.0 -> 57.8 mm
Other:
- board text added: "esp12 breakout rev1"
- board text removed: "RESET"

Commit message: move
Routing:
- net /RESET: track 61.8 -> 60.2 mm, vias 2 -> 0
